File: kicad/pcb/bully.kicad_sch (KiCad schematic)
At the start: 29 parts, among them J1 SM04B-SRSS-TB(LF)(SN), J2 Conn_01x04, U1 W25Q128JVS, U3 RP2040, U4 XC6206PxxxMR-Regulator_Linear, Y1 12MHz

Commit message: update ver num
Other:
- title: Bully2040 - MX/Alps -> Bully2040
Changed lines of the file:
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@@
   (paper "A4")
   (title_block
-    (title "Bully2040 - MX/Alps")
+    (title "Bully2040")
     (date "2023-06-23")
-    (rev "0.1")
+    (rev "0.2")
     (company "sporkus")
+    (comment 1 "adding alps and layout options")
   )
   (junction (at 205.74 62.23) (diameter 0) (color 0 0 0 0)
