File: kicad/pcb/key_matrix.kicad_sch (KiCad schematic)
At the start: 107 parts, among them SW1 SW_Push, SW10 SW_Push, SW11 SW_Push, SW12 SW_Push, SW13 SW_Push, SW14 SW_Push, SW15 SW_Push, SW16 SW_Push, SW17 SW_Push, SW18 SW_Push, SW19 SW_Push, SW2 SW_Push, SW20 SW_Push, SW21 SW_Push, SW22 SW_Push, SW23 SW_Push, SW24 SW_Push, SW25 SW_Push, SW26 SW_Push, SW27 SW_Push, SW28 SW_Push, SW29 SW_Push, SW3 SW_Push, SW30 SW_Push, SW31 SW_Push, SW32 SW_Push, SW33 SW_Push, SW34 SW_Push, SW35 SW_Push, SW36 SW_Push, SW37 SW_Push, SW38 SW_Push, SW39 SW_Push, SW4 SW_Push, SW40 SW_Push, SW41 SW_Push, SW42 SW_Push, SW43 SW_Push, SW44 SW_Push, SW45 SW_Push, SW5 SW_Push, SW54 RotaryEncoder_Switch, SW6 SW_Push, SW7 SW_Push, SW8 SW_Push, SW9 SW_Push

Commit message: update ver num
Other:
- title: Bully2040 - MX/Alps -> Bully2040
Changed lines of the file:
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@@
   (paper "A4")
   (title_block
-    (title "Bully2040 - MX/Alps")
+    (title "Bully2040")
     (date "2023-06-23")
-    (rev "0.1")
+    (rev "0.2")
     (company "sporkus")
+    (comment 1 "adding alps and layout options")
   )
   (junction (at 130.81 104.394) (diameter 0) (color 0 0 0 0)
